Commit message: URDF Corrections

File: src/mini_challenge2/urdf/puzzlebot.urdf (robot description, URDF)
Before this commit: robot puzzlebot, 5 links, 4 joints
Links:
- link base_link: geometry visual mesh filename=package://mini_challenge2/meshes/MCR2_puzzlebot_jetson_lida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
Joints:
- joint base_link_joint: origin xyz=0.0 0.0 0.05 rpy=0.0 0.0 0.0 -> xyz=0.0 0.0 0.065 rpy=0.0 0.0 0.0
- joint wheel_l_joint: origin xyz=0.052 0.095 -0.0025 rpy=0.0 0.0 0.0 -> xyz=0.052 0.095 -0.0020 rpy=0.0 0.0 0.0
- joint wheel_r_joint: origin xyz=0.052 -0.095 -0.0025 rpy=0.0 0.0 0.0 -> xyz=0.052 -0.095 -0.0020 rpy=0.0 0.0 0.0
